File: pcb/smart_battery.kicad_pcb (KiCad board)
At the start: 2 copper layers, 76.2 x 95.2 mm, 18 parts, among them J1 feather long, J10 feather short, J2 feather short, J3 feather long, J4 feather short, J5 feather long, J6 feather short, J7 feather long, J8 feather short, J9 feather long

Commit message: Added switches to power battery module from large battery
Parts:
- removed the REF** at (99.1, 27.9)
- removed the REF** at (99.1, 73.7)
- removed the REF** at (73.7, 118.1)
- removed the REF** at (27.9, 100.3)
- removed the REF** at (27.9, 118.1)
- removed the REF** at (73.7, 100.3)
- removed the REF** at (27.9, 94.0)
- added C1: C10uF, Capacitor_SMD:C_0805_2012Metric, F.Cu at (148.6, 88.9)
- added C2: C10uF, Capacitor_SMD:C_0805_2012Metric, F.Cu at (144.8, 95.2)
- added C3: C1uF, Capacitor_SMD:C_0805_2012Metric, F.Cu at (152.4, 100.3)
- added J11: Conn_01x05_RTC, Connector_PinHeader_2.54mm:PinHeader_1x05_P2.54mm_Vertical, F.Cu at (147.3, 48.3)
- added PS1: TSR_1-2450, Converter_DCDC:Converter_DCDC_TRACO_TSR-1_THT, F.Cu at (124.5, 36.8)
- added PS2: TEC_2-2411, TEC_2:TEC24811, F.Cu at (80.0, 81.3)
- added R1: R2k, Resistor_SMD:R_0805_2012Metric, F.Cu at (129.5, 104.1)
- added R2: R2k, Resistor_SMD:R_0805_2012Metric, F.Cu at (114.5, 100.3)
- added R3: R10k, Resistor_SMD:R_0805_2012Metric, F.Cu at (123.2, 109.2)
- added R4: R10k, Resistor_SMD:R_0805_2012Metric, F.Cu at (135.9, 106.7)
- added R5: 100K, Resistor_SMD:R_0805_2012Metric, F.Cu at (163.8, 66.0)
- added RP1: MP930-0.002-1, mp930:Caddock-MP930-0-0-Recommended_Land_Pattern_, F.Cu at (138.4, 47.0)
- added RP2: MP930-0.002-1, mp930:Caddock-MP930-0-0-Recommended_Land_Pattern_, F.Cu at (158.8, 44.5)
- added U1: SPX3819M5-L-3-3, Package_TO_SOT_SMD:SOT-23-5, F.Cu at (113.0, 85.1)
- added U1Batt1: LTC4151CS-2PBF, eec:Linear_Technology-LTC4151CS-2PBF-Level_B, F.Cu at (158.8, 53.3)
- added U2Solar1: LTC4151CS-2PBF, eec:Linear_Technology-LTC4151CS-2PBF-Level_B, F.Cu at (138.4, 54.6)
Connections:
- net /A0 renamed Net-(J7-Pad12)
- net /A1 renamed Net-(J7-Pad11)
- net /A2 renamed Net-(J7-Pad10)
- net /F0 renamed Net-(J8-Pad3)
- net /F1 renamed Net-(J8-Pad4)
- net /F2 renamed Net-(J8-Pad5)
- net /F3 renamed Net-(J8-Pad6)
- net /F4 renamed Net-(J8-Pad7)
- net /F5 renamed Net-(J8-Pad8)
- net /F6 renamed Net-(J8-Pad9)
- net /VUSB renamed Net-(J8-Pad10)
- J1 pad 1: (no net) -> Net-(J1-Pad1)
- J1 pad 10: (no net) -> /VSSO
- J1 pad 11: (no net) -> /THBAT
- J1 pad 12: (no net) -> /THHTR
- J1 pad 13: (no net) -> GND
- J1 pad 14: (no net) -> /AREF
- J1 pad 15: (no net) -> +3V3
- J1 pad 16: (no net) -> /~RST
- J1 pad 2: (no net) -> /TX
- J1 pad 3: (no net) -> /RX
- J1 pad 4: (no net) -> /MISO
- J1 pad 5: (no net) -> /MOSI
- J1 pad 6: (no net) -> /SCK
- J1 pad 7: (no net) -> /A5
- J1 pad 8: (no net) -> /A4
- J1 pad 9: (no net) -> /VSPO
- J10 pad 1: (no net) -> Net-(J10-Pad1)
- J10 pad 10: (no net) -> Net-(J10-Pad10)
- J10 pad 11: (no net) -> Net-(J10-Pad11)
- J10 pad 12: (no net) -> Net-(J10-Pad12)
- J10 pad 2: (no net) -> Net-(J10-Pad2)
- J10 pad 3: (no net) -> Net-(J10-Pad3)
- J10 pad 4: (no net) -> Net-(J10-Pad4)
- J10 pad 5: (no net) -> Net-(J10-Pad5)
- J10 pad 6: (no net) -> Net-(J10-Pad6)
- J10 pad 7: (no net) -> Net-(J10-Pad7)
- J10 pad 8: (no net) -> Net-(J10-Pad8)
- J10 pad 9: (no net) -> Net-(J10-Pad9)
- J2 pad 1: (no net) -> /SDA
- J2 pad 10: (no net) -> +5V
- J2 pad 11: (no net) -> /EN
- J2 pad 12: (no net) -> /VBAT
- J2 pad 2: (no net) -> /SCL
- J2 pad 3: (no net) -> /SUSET
- J2 pad 4: (no net) -> /PSET
- J2 pad 5: (no net) -> /PUSET
- J2 pad 6: (no net) -> /ENCS
- J2 pad 7: (no net) -> /SSET
- J2 pad 8: (no net) -> /HTEN
- J2 pad 9: (no net) -> /VPIN
- J3 pad 1: (no net) -> Net-(J3-Pad1)
- J3 pad 10: (no net) -> Net-(J3-Pad10)
- J3 pad 11: (no net) -> Net-(J3-Pad11)
- J3 pad 12: (no net) -> Net-(J3-Pad12)
- J3 pad 13: (no net) -> GND
- J3 pad 14: (no net) -> Net-(J3-Pad14)
- J3 pad 15: (no net) -> +3V3
- J3 pad 16: (no net) -> /~RST
- J3 pad 2: (no net) -> Net-(J3-Pad2)
- J3 pad 3: (no net) -> Net-(J3-Pad3)
- J3 pad 4: (no net) -> Net-(J3-Pad4)
- J3 pad 5: (no net) -> Net-(J3-Pad5)
- J3 pad 6: (no net) -> Net-(J3-Pad6)
- J3 pad 7: (no net) -> Net-(J3-Pad7)
- J3 pad 8: (no net) -> Net-(J3-Pad8)
- J3 pad 9: (no net) -> Net-(J3-Pad9)
- J4 pad 1: (no net) -> Net-(J4-Pad1)
- J4 pad 10: (no net) -> /HTEN
- J4 pad 11: (no net) -> Net-(J4-Pad11)
- J4 pad 12: (no net) -> Net-(J4-Pad12)
- J4 pad 2: (no net) -> Net-(J4-Pad2)
- J4 pad 3: (no net) -> Net-(J4-Pad3)
- J4 pad 4: (no net) -> Net-(J4-Pad4)
- J4 pad 5: (no net) -> Net-(J4-Pad5)
- J4 pad 6: (no net) -> Net-(J4-Pad6)
- J4 pad 7: (no net) -> Net-(J4-Pad7)
- J4 pad 8: (no net) -> Net-(J4-Pad8)
- J4 pad 9: (no net) -> Net-(J4-Pad9)
- J5 pad 1: (no net) -> /FREE
- J5 pad 10: (no net) -> Net-(J5-Pad10)
- J5 pad 11: (no net) -> Net-(J5-Pad11)
- J5 pad 12: (no net) -> Net-(J5-Pad12)
- J5 pad 13: (no net) -> GND
- J5 pad 14: (no net) -> Net-(J5-Pad14)
- J5 pad 15: (no net) -> /Eth3.3
- J5 pad 16: (no net) -> /~RST
- J5 pad 2: (no net) -> Net-(J5-Pad2)
- J5 pad 3: (no net) -> Net-(J5-Pad3)
- J5 pad 4: (no net) -> /MISO
- J5 pad 5: (no net) -> /MOSI
- J5 pad 6: (no net) -> /SCK
- J5 pad 7: (no net) -> Net-(J5-Pad7)
- J5 pad 8: (no net) -> Net-(J5-Pad8)
- J5 pad 9: (no net) -> Net-(J5-Pad9)
- J6 pad 1: (no net) -> Net-(J6-Pad1)
- J6 pad 10: (no net) -> Net-(J6-Pad10)
- J6 pad 11: (no net) -> Net-(J6-Pad11)
- J6 pad 12: (no net) -> Net-(J6-Pad12)
- J6 pad 2: (no net) -> Net-(J6-Pad2)
- J6 pad 3: (no net) -> Net-(J6-Pad3)
- J6 pad 4: (no net) -> Net-(J6-Pad4)
- J6 pad 5: (no net) -> Net-(J6-Pad5)
- J6 pad 6: (no net) -> /CS
- J6 pad 7: (no net) -> Net-(J6-Pad7)
- J6 pad 8: (no net) -> Net-(J6-Pad8)
- J6 pad 9: (no net) -> Net-(J6-Pad9)
- J7 pad 1: /FREE -> Net-(J7-Pad1)
- J7 pad 13: GND -> Net-(J7-Pad13)
- J7 pad 14: /AREF -> Net-(J7-Pad14)
- J7 pad 15: +3V3 -> Net-(J7-Pad15)
- J7 pad 2: /TX -> Net-(J7-Pad2)
- J7 pad 3: /RX -> Net-(J7-Pad3)
- J7 pad 4: /MISO -> Net-(J7-Pad4)
- J7 pad 5: /MOSI -> Net-(J7-Pad5)
- J7 pad 6: /SCK -> /SOUT
- J7 pad 7: /A5 -> +5V
- J7 pad 8: /A4 -> /SUSET
- J7 pad 9: /A3 -> /SSET
- J8 pad 1: /SDA -> Net-(J8-Pad1)
- J8 pad 11: /EN -> Net-(J8-Pad11)
- J8 pad 12: /VBAT -> Net-(J8-Pad12)
- J8 pad 2: /SCL -> Net-(J8-Pad2)
- J9 pad 1: (no net) -> Net-(J9-Pad1)
- J9 pad 10: (no net) -> Net-(J9-Pad10)
- J9 pad 11: (no net) -> Net-(J9-Pad11)
- J9 pad 12: (no net) -> Net-(J9-Pad12)
- J9 pad 13: (no net) -> Net-(J9-Pad13)
- J9 pad 14: (no net) -> Net-(J9-Pad14)
- J9 pad 15: (no net) -> Net-(J9-Pad15)
- J9 pad 16: (no net) -> /~RST
- J9 pad 2: (no net) -> Net-(J9-Pad2)
- J9 pad 3: (no net) -> Net-(J9-Pad3)
- J9 pad 4: (no net) -> Net-(J9-Pad4)
- J9 pad 5: (no net) -> Net-(J9-Pad5)
- J9 pad 6: (no net) -> /POUT
- J9 pad 7: (no net) -> +5V
- J9 pad 8: (no net) -> /PUSET
- J9 pad 9: (no net) -> /PSET

Commit message: Moving to a feather symbol library
Parts:
- removed C1, C2: C10uF, Capacitor_SMD:C_0805_2012Metric
- removed C3: C1uF, Capacitor_SMD:C_0805_2012Metric
- removed J1, J3, J5, J7, J9: feather long, Connector_PinHeader_2.54mm:PinHeader_1x16_P2.54mm_Vertical
- removed J10, J2, J4, J6, J8: feather short, Connector_PinHeader_2.54mm:PinHeader_1x12_P2.54mm_Vertical
- removed J11: Conn_01x05_RTC, Connector_PinHeader_2.54mm:PinHeader_1x05_P2.54mm_Vertical
- removed PS1: TSR_1-2450, Converter_DCDC:Converter_DCDC_TRACO_TSR-1_THT
- removed PS2: TEC_2-2411, TEC_2:TEC24811
- removed R1, R2: R2k, Resistor_SMD:R_0805_2012Metric
- removed R3, R4: R10k, Resistor_SMD:R_0805_2012Metric
- removed R5: 100K, Resistor_SMD:R_0805_2012Metric
- removed REF**: MountingHole_2.7mm_M2.5, MountingHole:MountingHole_2.7mm_M2.5
- removed RP1, RP2: MP930-0.002-1, mp930:Caddock-MP930-0-0-Recommended_Land_Pattern_
- removed U1: SPX3819M5-L-3-3, Package_TO_SOT_SMD:SOT-23-5
- removed U1Batt1, U2Solar1: LTC4151CS-2PBF, eec:Linear_Technology-LTC4151CS-2PBF-Level_B
Other:
- board outline removed
- board text removed: "3V3"
- board text removed: "A0"
- board text removed: "A1"
- board text removed: "A2"
- board text removed: "A3"
- board text removed: "A4"
- board text removed: "A5"
- board text removed: "AREF"
- board text removed: "EN"
- board text removed: "F0"
- board text removed: "F1"
- board text removed: "F2"
- board text removed: "F3"
- board text removed: "F4"
- board text removed: "F5"
- board text removed: "F6"
- board text removed: "FREE"
- board text removed: "GND"
- board text removed: "MISO"
- board text removed: "MOSI"
- board text removed: "RX"
- board text removed: "SCK"
- board text removed: "SCL"
- board text removed: "SDA"
- board text removed: "TX"
- board text removed: "VBAT"
- board text removed: "VUSB"
- board text removed: "~RST"

Commit message: Post review changes
Parts:
- added C1: C10uF, Capacitor_SMD:C_0805_2012Metric, F.Cu at (100.0, 109.3)
- added C2: C10uF, Capacitor_SMD:C_0805_2012Metric, F.Cu at (83.0, 109.3)
- added C3: C1uF, Capacitor_SMD:C_0805_2012Metric, F.Cu at (96.6, 109.3)
- added J11: Conn_01x05_RTC, Connector_PinHeader_2.54mm:PinHeader_1x05_P2.54mm_Vertical, F.Cu at (196.1, 51.6)
- added J12: Conn_HtrTh, Connector_Molex:Molex_KK-254_AE-6410-02A_1x02_P2.54mm_Vertical, F.Cu at (185.8, 83.2)
- added J13: Conn_BattTh, Connector_Molex:Molex_KK-254_AE-6410-02A_1x02_P2.54mm_Vertical, F.Cu at (196.1, 67.0)
- added JM1: RockBLOCK Modem, Connector_Molex:Molex_KK-254_AE-6410-04A_1x04_P2.54mm_Vertical, F.Cu at (146.1, 77.5)
- added JM2: I2C Connector, Connector_Molex:Molex_KK-254_AE-6410-04A_1x04_P2.54mm_Vertical, F.Cu at (185.8, 76.4)
- added JP1: SolarIn, eec:7.5mm_screw_conn_1x2, F.Cu at (184.2, 21.6)
- added JP2: SolarOut, eec:7.5mm_screw_conn_1x3, F.Cu at (170.2, 47.0)
- added JP3: BatteryIn, eec:7.5mm_screw_conn_1x2, F.Cu at (184.2, 41.9)
- added JP4: BatteryOut, eec:7.5mm_screw_conn_1x3, F.Cu at (170.2, 21.6)
- added PS1: TSR_1-2450, Converter_DCDC:Converter_DCDC_TRACO_TSR-1_THT, F.Cu at (114.3, 81.3)
- added PS2: TEC_2-2411, TEC_2:TEC24811, F.Cu at (125.7, 26.7)
- added Q1: MMBT5551L, Package_TO_SOT_SMD:SOT-23, F.Cu at (180.3, 86.7)
- added Q2: MMBT5551L, Package_TO_SOT_SMD:SOT-23, F.Cu at (206.9, 55.2)
- added R1: R2k, Resistor_SMD:R_0805_2012Metric, F.Cu at (86.4, 109.3)
- added R2: R2k, Resistor_SMD:R_0805_2012Metric, F.Cu at (106.9, 109.3)
- added R3: R10k, Resistor_SMD:R_0805_2012Metric, F.Cu at (89.8, 109.3)
- added R4: R10k, Resistor_SMD:R_0805_2012Metric, F.Cu at (93.2, 109.3)
- added R5: 100K, Resistor_SMD:R_0805_2012Metric, F.Cu at (117.1, 109.3)
- added R6: R68k, Resistor_SMD:R_0805_2012Metric, F.Cu at (113.7, 109.3)
- added R7: 5.1K, Resistor_SMD:R_0805_2012Metric, F.Cu at (103.4, 109.3)
- added R8: 15K, Resistor_SMD:R_0805_2012Metric, F.Cu at (134.3, 109.1)
- added R9: 1K, Resistor_SMD:R_0805_2012Metric, F.Cu at (110.3, 109.3)
- added RP1: MP930-0.002-1, mp930:Caddock-MP930-0-0-Recommended_Land_Pattern_, F.Cu at (133.3, 41.9)
- added RP2: MP930-0.002-1, mp930:Caddock-MP930-0-0-Recommended_Land_Pattern_, F.Cu at (203.4, 55.2)
- added U1: SPX3819M5-L-3-3, Package_TO_SOT_SMD:SOT-23-5, F.Cu at (207.1, 51.6)
- added U10: FEATHER_M0_ADALOGGER, SMARTBATT:MODULE_FEATHER_M0_BASIC_PROTO, F.Cu at (50.8, 106.7)
- added U11: FEATHERWING_POWER_RELAY, SMARTBATT:MODULE_FEATHER_POWER_RELAY, F.Cu at (49.5, 81.3)
- added U12: FEATHERWING_ETHERNET, SMARTBATT:MODULE_FEATHER_ETHERNET_MODULE, F.Cu at (90.2, 44.5)
- added U13: FEATHERWING_MINI_RELAY, SMARTBATT:MODULE_FEATHER_MINI_RELAY, F.Cu at (49.5, 55.9)
- added U14: FEATHERWING_MINI_RELAY, SMARTBATT:MODULE_FEATHER_MINI_RELAY, F.Cu at (48.3, 30.5)
- added U1Batt1: LTC4151CS-2PBF, eec:Linear_Technology-LTC4151CS-2PBF-Level_B, B.Cu at (130.8, 61.0)
- added U2Solar1: LTC4151CS-2PBF, eec:Linear_Technology-LTC4151CS-2PBF-Level_B, F.Cu at (153.7, 54.6)

Commit message: Laying out board
Parts:
- C1, C2, C3, Q1, Q2, R1, R2, R3, R4, R5, R6, R7, R8, R9, U1, U2Solar1: moved to B.Cu
- JM1: footprint Connector_Molex:Molex_KK-254_AE-6410-04A_1x04_P2.54mm_Vertical -> Connector_Molex:Molex_KK-254_AE-6410-06A_1x06_P2.54mm_Vertical
- U11: value FEATHERWING_POWER_RELAY -> FEATHERWING_HEATER_RELAY
- moved Q2 125.6 mm to (91.7, 105.0)
- moved U1 119.3 mm to (89.2, 34.1), turned to 180 degrees
- moved RP2 99.9 mm to (114.3, 100.3), turned to 180 degrees
- moved J13 97.2 mm to (110.5, 113.0)
- moved JM2 96.0 mm to (94.0, 48.3), turned to 180 degrees
- moved JP4 93.9 mm to (123.2, 102.9), turned to 180 degrees
- moved J12 89.3 mm to (101.6, 113.0)
- moved J11 87.0 mm to (109.2, 47.0), turned to 270 degrees
- moved C3 87.0 mm to (89.2, 22.7)
- moved JP3 83.6 mm to (123.2, 99.1)
- moved Q1 83.3 mm to (98.1, 100.0)
- moved C2 81.8 mm to (89.2, 27.8)
- moved C1 80.2 mm to (94.2, 29.4), turned to 90 degrees
- moved R5 78.6 mm to (94.2, 34.1), turned to 90 degrees
- moved JP1 74.0 mm to (123.2, 63.5)
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Connections:
- net /A4 renamed /48VEN
- net /EN renamed Net-(U10-PadP2_2)
- JM1 pad 3: /RX -> /RBRX
- JM1 pad 4: /TX -> /RBTX
- JP2 pad 2: GND -> /SOLPWR
- U10 pad P1_10: /VSSO -> /RBRX
- U10 pad P1_7: /A5 -> /RBEN
- U10 pad P1_9: /VSPO -> /RBTX
- U12 pad P2_3: +5V -> Net-(U12-PadP2_3)
- U14 pad P2_1: /POUT -> Net-(U14-PadP2_1)
- U14 pad P2_2: Net-(U14-PadP2_2) -> /POUT

Commit message: First board layout done
Routing:
- net GND: track 0.00 -> 493.2 mm
- net +5V: track 0.00 -> 195.5 mm
- net /SDA: track 0.00 -> 141.0 mm
- net /~RST: track 0.00 -> 138.0 mm
- net /SCL: track 0.00 -> 134.9 mm
- net +3V3: track 0.00 -> 133.9 mm
- net /ENCS: track 0.00 -> 119.3 mm
- net /VPIN: track 0.00 -> 107.1 mm, vias 0 -> 1
- net /MISO: track 0.00 -> 102.5 mm
- net /MOSI: track 0.00 -> 102.5 mm
- net /SCK: track 0.00 -> 102.1 mm
- net /THBAT: track 0.00 -> 93.6 mm
- net /THHTR: track 0.00 -> 76.9 mm
- net /PUSET: track 0.00 -> 68.6 mm
- net /PSET: track 0.00 -> 66.4 mm
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